Commit message: Change_ removed links to Adafruit and Teensy

File: diffbot_description/urdf/diffbot.urdf.xacro (robot description, xacro)
@@ -50,4 +50,7 @@
                    enable_gpu="${sensor_prop['laser']['enable_gpu']}">
   </xacro:laser>
+  <xacro:imu_sensor parent_link="base_link"
+                   sensor_prop="${sensor_prop}">
+  </xacro:imu_sensor>
   <!-- Gazebo -->
   <xacro:gazebo_ros_control robotNamespace="/diffbot">

File: diffbot_description/urdf/include/common_sensors.xacro (robot description, xacro)
@@ -175,5 +175,5 @@
   </gazebo>
 </xacro:macro>
-<xacro:macro name="imu_sensor" params=" *joint_origin parent_link sensor_prop">
+<xacro:macro name="imu_sensor" params="parent_link sensor_prop">
   <xacro:property name="mesh"
      value="${sensor_prop['imu']['mesh']}"/>
@@ -223,6 +223,7 @@
   </gazebo>
   <joint name="imu_joint" type="fixed">
-    <axis xyz="0 1 0" />
-    <xacro:insert_block name="joint_origin" />
+    <!-- SBR:   <xacro:insert_block name="joint_origin" />-->
+    <!--<origin xyz="${sensor_prop['imu']['dx']} ${sensor_prop['imu']['dy']} ${sensor_prop['imu']['dz']}" rpy="0 0 0"/>-->
+    <origin xyz="0 0 0" rpy="0 0 0"/>
     <parent link="${parent_link}"/>
     <child link="imu_link"/>

Commit message: Add raspi camera to urdf and gmapping launch file

File: diffbot_description/urdf/diffbot.urdf.xacro (robot description, xacro)
@@ -53,4 +53,7 @@
                    sensor_prop="${sensor_prop}">
   </xacro:imu_sensor>
+  <xacro:camera_sensor parent_link="base_link"
+                   sensor_prop="${sensor_prop}">
+  </xacro:camera_sensor>
   <!-- Gazebo -->
   <xacro:gazebo_ros_control robotNamespace="/diffbot">

File: diffbot_description/urdf/include/common_sensors.xacro (robot description, xacro)
@@ -91,4 +91,5 @@
   </gazebo>
 </xacro:macro>
+<!--
 <xacro:macro name="camera_sensor" params=" *joint_origin parent_link sensor_prop visualize mesh:='' ">
   <link name="camera_link">
@@ -151,7 +152,4 @@
         <noise>
           <type>gaussian</type>
-          <!-- Noise is sampled independently per pixel on each frame.
-                That pixel's noise value is added to each of its color
-                channels, which at that point lie in the range [0,1]. -->
           <mean>0.0</mean>
           <stddev>0.007</stddev>
@@ -174,4 +172,59 @@
     </sensor>
   </gazebo>
+</xacro:macro>
+-->
+<xacro:macro name="camera_sensor" params="parent_link sensor_prop visualize:='true' mesh:='' ">
+    <joint name="camera_joint" type="fixed">
+        <parent link="${parent_link}"/>
+        <child link="camera_link"/>
+        <origin xyz="0.12 0 0.02" rpy="0 0 0"/>
+        <axis xyz="0 0 0" />
+    </joint>
+    <link name="camera_link">
+        <visual>
+            <geometry>
+                <box size="0.010 0.03 0.03"/>
+            </geometry>
+            <material name="black"/>
+        </visual>
+        <visual>
+            <origin xyz="0 0 -0.01" rpy="0 0 0"/>
+            <geometry>
+                <cylinder radius="0.004" length="0.01"/>
+            </geometry>
+            <material name="black"/>
+        </visual>
+    </link>
+   <!--
+    <joint name="camera_optical_joint" type="fixed">
+        <parent link="camera_link"/>
+        <child link="camera_link_optical"/>
+        <origin xyz="0 0 0" rpy="${-pi/2} 0 ${-pi/2}"/>
+    </joint>
+    <link name="camera_link_optical"></link>
+    -->
+    <gazebo reference="camera_link">
+        <material>Gazebo/Black</material>
+        <sensor name="camera" type="camera">
+            <pose> 0 0 0 0 0 0 </pose>
+            <visualize>true</visualize>
+            <update_rate>10</update_rate>
+            <camera>
+                <horizontal_fov>1.089</horizontal_fov>
+                <image>
+                    <format>R8G8B8</format>
+                    <width>640</width>
+                    <height>480</height>
+                </image>
+                <clip>
+                    <near>0.05</near>
+                    <far>8.0</far>
+                </clip>
+            </camera>
+            <plugin name="camera_controller" filename="libgazebo_ros_camera.so">
+                <frame_name>camera_link_optical</frame_name>
+            </plugin>
+        </sensor>
+    </gazebo>
 </xacro:macro>
 <xacro:macro name="imu_sensor" params="parent_link sensor_prop">

Commit message: Updatred Config + URDF + Xacro to Real SBR Robot

File: diffbot_description/urdf/diffbot.urdf.xacro (robot description, xacro)
@@ -9,6 +9,6 @@
   <xacro:property name="caster_wheel_yaml" value="$(find ${package_name})/config/${robot_name}/caster_wheel.yaml" />
   <xacro:property name="caster_wheel_props" value="${xacro.load_yaml(caster_wheel_yaml)}"/>
-  <xacro:property name="front_wheel_yaml" value="$(find ${package_name})/config/${robot_name}/front_wheel.yaml" />
-  <xacro:property name="front_wheel_props" value="${xacro.load_yaml(front_wheel_yaml)}"/>
+  <xacro:property name="rear_wheel_yaml" value="$(find ${package_name})/config/${robot_name}/back_wheel.yaml" />
+  <xacro:property name="rear_wheel_props" value="${xacro.load_yaml(rear_wheel_yaml)}"/>
   <xacro:property name="motor_yaml" value="$(find ${package_name})/config/${robot_name}/motor.yaml" />
   <xacro:property name="motor_props" value="${xacro.load_yaml(motor_yaml)}"/>
@@ -18,5 +18,5 @@
   <xacro:property name="sensor_prop" value="${xacro.load_yaml(sensor_yaml)}"/>
   <!-- Footprint link -->
-  <xacro:footprint wheel_props="${front_wheel_props}" />
+  <xacro:footprint wheel_props="${rear_wheel_props}" />
   <!-- Base link -->
   <xacro:base base_prop="${base_props}" mesh="${base_props['base']['mesh']}" >
@@ -24,14 +24,14 @@
   </xacro:base>
   <!-- Back Caster Wheel -->
-  <xacro:caster_wheel prefix="rear" reflect="-1"
+  <xacro:caster_wheel prefix="front" reflect="-1"
                       wheel_props="${caster_wheel_props}">
   </xacro:caster_wheel>
   <!-- Front Wheels -->
-  <xacro:wheel prefix="front_right" reflect="-1"
-                      wheel_props="${front_wheel_props}"
+  <xacro:wheel prefix="rear_right" reflect="-1"
+                      wheel_props="${rear_wheel_props}"
                       base_props="${base_props}" >
   </xacro:wheel>
-  <xacro:wheel prefix="front_left" reflect="1"
-                      wheel_props="${front_wheel_props}"
+  <xacro:wheel prefix="rear_left" reflect="1"
+                      wheel_props="${rear_wheel_props}"
                       base_props="${base_props}" >
   </xacro:wheel>

File: diffbot_description/urdf/include/common_macros.urdf.xacro (robot description, xacro)
@@ -165,5 +165,5 @@
     <xacro:if value="${mesh != '' }" >
       <visual>
-        <xacro:insert_block name="origin" />
+        <origin xyz="0.04 0.0 0.017" rpy="1.57 0.0 0.0"/>
         <geometry>
           <!-- The folder path get a folder_name global parameter -->
@@ -175,5 +175,5 @@
           </xacro:if>
         </geometry>
-        <material name="white" />
+        <material name="dark_grey" />
       </visual>
     </xacro:if>
@@ -184,5 +184,5 @@
           <box size="${base_prop['base']['x_size']} ${base_prop['base']['y_size']} ${base_prop['base']['z_size']}"/>
         </geometry>
-        <material name="white" />
+        <material name="red" />
       </visual>
     </xacro:if>

File: diffbot_description/urdf/include/common_sensors.xacro (robot description, xacro)
@@ -178,5 +178,5 @@
         <parent link="${parent_link}"/>
         <child link="camera_link"/>
-        <origin xyz="0.12 0 0.02" rpy="0 0 0"/>
+        <origin xyz="0.12 0 0.1" rpy="0 0 0"/>
         <axis xyz="0 0 0" />
     </joint>
@@ -189,5 +189,5 @@
         </visual>
         <visual>
-            <origin xyz="0 0 -0.01" rpy="0 0 0"/>
+            <origin xyz="0.01 0 0.0" rpy="0 0 0"/>
             <geometry>
                 <cylinder radius="0.004" length="0.01"/>
@@ -234,14 +234,14 @@
     <xacro:if value="${mesh != '' }" >
       <visual>
-        <origin xyz="0 0 0" rpy="0 0 0"/>
+        <origin xyz="-0.01 0.05 0.13" rpy="0 0 0"/>
         <geometry>
           <mesh filename="package://${package_name}/meshes/sensors/${mesh}" scale="${sensor_prop['imu']['scale']}" />
         </geometry>
-        <material name="dark_grey"/>
+        <material name="blue"/>
       </visual>
     </xacro:if>
     <xacro:if value="${mesh == '' }" >
       <visual>
-        <origin xyz="0 0 0" rpy="0 0 0"/>
+        <origin xyz="0.1 0 0" rpy="0 0 0"/>
         <geometry>
           <cylinder radius="${sensor_prop['imu']['radius']}" length="${sensor_prop['imu']['length']}"/>

File: diffbot_description/urdf/include/diffbot_caster_macro.urdf.xacro (robot description, xacro)
@@ -28,8 +28,8 @@
           <origin xyz="0 0 ${-wheel_props['base']['size']['z']/2.0}" rpy="0 0 0" />
           <geometry>
-            <xacro:if value="${scale != '' }" >
-              <mesh filename="package://${package_name}/meshes/${robot_name}/${wheel_props['base']['mesh']}" scale="${scale}"/>
+            <xacro:if value="${wheel_props['scale'] != '' }" >
+              <mesh filename="package://${package_name}/meshes/${robot_name}/${wheel_props['base']['mesh']}" scale="${wheel_props['scale']}"/>
             </xacro:if>
-            <xacro:if value="${scale == '' }" >
+            <xacro:if value="${wheel_props['scale'] == '' }" >
               <mesh filename="package://${package_name}/meshes/${robot_name}/${wheel_props['base']['mesh']}" />
             </xacro:if>
@@ -78,8 +78,8 @@
           <origin xyz="0 0 ${-wheel_props['hub']['size']['z']/2.0}" rpy="0 0 0" />
           <geometry>
-            <xacro:if value="${scale != '' }" >
-              <mesh filename="package://${package_name}/meshes/${robot_name}/${wheel_props['hub']['mesh']}" scale="${scale}"/>
+            <xacro:if value="${wheel_props['scale'] != '' }" >
+              <mesh filename="package://${package_name}/meshes/${robot_name}/${wheel_props['hub']['mesh']}" scale="${wheel_props['scale']}"/>
             </xacro:if>
-            <xacro:if value="${scale == '' }" >
+            <xacro:if value="${wheel_props['scale'] == '' }" >
               <mesh filename="package://${package_name}/meshes/${robot_name}/${wheel_props['hub']['mesh']}" />
             </xacro:if>
@@ -127,8 +127,8 @@
           <origin xyz="0 0 0" rpy="0 0 0" />
           <geometry>
-            <xacro:if value="${scale != '' }" >
-              <mesh filename="package://${package_name}/meshes/${robot_name}/${wheel_props['wheel']['mesh']}" scale="${scale}"/>
+            <xacro:if value="${wheel_props['scale'] != '' }" >
+              <mesh filename="package://${package_name}/meshes/${robot_name}/${wheel_props['wheel']['mesh']}" scale="${wheel_props['scale']}"/>
             </xacro:if>
-            <xacro:if value="${scale == '' }" >
+            <xacro:if value="${wheel_props['scale'] == '' }" >
               <mesh filename="package://${package_name}/meshes/${robot_name}/${wheel_props['wheel']['mesh']}" />
             </xacro:if>
